File: electrical/source/weather-station.kicad_sch (KiCad schematic)
At the start: 0 parts

Commit message: KiCad, finished the schematic for the Raspberry Pi
Parts:
- added A1: Raspberry_Pi_3_B+, symbol weather-station:Raspberry_Pi_3_B+
- added A2: Adafruit_MCP9808_5027, symbol weather-station:Adafruit_MCP9808_5027
- added D1: LED, symbol Device:LED
- added R1: 147 Ω, symbol Device:R
- added SW1: Rain_Sensor_MS-WH-SP-RG, symbol weather-station:Rain_Sensor_MS-WH-SP-RG
Connections:
- new net: A1. (USB_2), A2. (VIN) (x4)
- new net: A1. (USB_2), R1.1
- new net: D1.2 (A), R1.2
- new net: A1. (USB_2), D1.1 (K)
- new net: A1. (USB_2), SW1. (6) (x2)
- no-connect marks 0 -> 45
